Commit message: New objective test done

File: assets/robot/urdf/fr3_robotiq.urdf (robot description, URDF)
Before this commit: robot fr3, 24 links, 23 joints
Links:
- added link wrist_camera, mass 0.108; visual box size=0.1245 0.0305 0.0265
Joints:
- added joint wrist_camera_joint: type fixed, parent fr3_gripper, child wrist_camera, origin xyz=-0.068245 0.041394 0.029241 rpy=-0.297255482 0.00901527262 -1.62271473

File: assets/robot/urdf/fr3_robotiq_rigid.urdf (robot description, URDF)
Before this commit: robot fr3, 24 links, 23 joints
Links:
- added link wrist_camera, mass 0.108; visual box size=0.1245 0.0305 0.0265
Joints:
- added joint wrist_camera_joint: type fixed, parent fr3_gripper, child wrist_camera, origin xyz=-0.068245 0.041394 0.029241 rpy=-0.297255482 0.00901527262 -1.62271473
